Commit message: Fix URDF and CMakeLists

File: urdf/cobblestone.urdf (robot description, URDF)
Before this commit: robot wood, 1 links, 0 joints
Links:
- link base_link: geometry collision mesh filename=package://gerard-bauzil/cobblestone.dae; visual mesh filename=package://gerard-bauzil/cobblestone.dae
