Commit message: Rename gerard-bauzil -> gerard_bauzil in urdf/staircases_koroibot.urdf.

File: urdf/staircases_koroibot.urdf (robot description, URDF)
Before this commit: robot staircase, 1 links, 0 joints
Links:
- link base_link: geometry collision mesh filename=package://gerard_bauzil/staircases_koroibot_hr.dae; visual mesh filename=package://gerard_bauzil/staircases_koroibot_hr.dae
