Commit message: Fix axis of visual tag on cardboard_box

File: urdf/cardboard_box.urdf (robot description, URDF)
Before this commit: robot cardboard_box, 3 links, 2 joints
Links:
- link tag36_11_00002: geometry visual box size=0.06 0.06 0.002
Joints:
- joint tag36_11_00002_joint: origin xyz=-0.056  0.0195 0.01 -> xyz=-0.056  0.0195 0.01 rpy=1.5707963267948966 0 3.141592653589793
