Commit message: Add visual tag on pedestal table.

File: urdf/pedestal_table.urdf (robot description, URDF)
Before this commit: robot table, 1 links, 0 joints
Links:
- added link tag36_11_00001; visual box size=0.06 0.06 0.002
Joints:
- added joint tag36_11_00001_joint: type fixed, parent base_link, child tag36_11_00001, origin xyz=0.079 0.1255 1.095 rpy=0 0 -1.5707963267948966
