Commit message: [table] Put table on a fixed joint to make it movable.

File: urdf/table_140_70_73.urdf (robot description, URDF)
Before this commit: robot table, 1 links, 0 joints
Links:
- added link table_link, mass 2.2; collision box size=.02 .02 .72; collision box size=.02 .02 .72
- added link tag36_11_00004; visual box size=0.0635 0.0635 0.002
- added link tag36_11_00005; visual box size=0.0635 0.0635 0.002
- link base_link: mass 2.2 -> None; geometry 
Joints:
- added joint table_joint: type fixed, parent base_link, child table_link, origin xyz=0 0 0.005
- added joint tag36_11_00004_joint: type fixed, parent base_link, child tag36_11_00004, origin xyz=0.647 -0.0685 0.73
- added joint tag36_11_00005_joint: type fixed, parent base_link, child tag36_11_00005, origin xyz=0.123 -0.287 0.73

Commit message: [Table] Add tolerance for collision (2cm).

File: urdf/table_140_70_73.urdf (robot description, URDF)
Before this commit: robot table, 4 links, 3 joints
Links:
- link table_link: geometry collision box size=.02 .02 .72; collision box size=.02 .02 .72

Commit message: [table] Fix position of tags

File: urdf/table_140_70_73.urdf (robot description, URDF)
Before this commit: robot table, 4 links, 3 joints
Joints:
- joint tag36_11_00004_joint: origin xyz=0.647 -0.0685 0.73 -> xyz=0.647 -0.0685 0.73 rpy=0 0 -1.5707963267948966
- joint tag36_11_00005_joint: origin xyz=0.123 -0.287 0.73 -> xyz=0.123 -0.287 0.73 rpy=0 0 -1.5707963267948966

Commit message: [table] Attach tag to table_link, not base_link

File: urdf/table_140_70_73.urdf (robot description, URDF)
Before this commit: robot table, 4 links, 3 joints
Joints:
- joint tag36_11_00004_joint: parent base_link -> table_link
- joint tag36_11_00005_joint: parent base_link -> table_link
