Commit message: [Plank_of_wood] Resize collision geometry to fit visual geometry.

File: urdf/plank_of_wood1.urdf (robot description, URDF)
Before this commit: robot plank_of_wood1, 5 links, 4 joints
Links:
- link base_link: geometry collision box size=0.203 0.116 0.043; visual box size=0.203 0.116 0.043

File: urdf/plank_of_wood2.urdf (robot description, URDF)
Before this commit: robot plank_of_wood2, 5 links, 4 joints
Links:
- link base_link: geometry collision box size=0.203 0.116 0.043; visual box size=0.203 0.116 0.043

File: urdf/plank_of_wood3.urdf (robot description, URDF)
Before this commit: robot plank_of_wood3, 5 links, 4 joints
Links:
- link base_link: geometry collision box size=0.203 0.116 0.043; visual box size=0.203 0.116 0.043

File: urdf/plank_of_wood4.urdf (robot description, URDF)
Before this commit: robot plank_of_wood4, 5 links, 4 joints
Links:
- link base_link: geometry collision box size=0.203 0.116 0.043; visual box size=0.203 0.116 0.043

Commit message: Add AprilTags on boxes and tables

File: urdf/plank_of_wood1.urdf (robot description, URDF)
Before this commit: robot plank_of_wood1, 5 links, 4 joints
Links:
- link tag36_11_00010: geometry visual mesh filename=package://gerard_bauzil/meshes/apriltag_36h11/tag36_11_0001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 scale=0.075 0.075 1.
- link tag36_11_00011: geometry visual mesh filename=package://gerard_bauzil/meshes/apriltag_36h11/tag36_11_0001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 scale=0.075 0.075 1.
- link tag36_11_00012: geometry visual mesh filename=package://gerard_bauzil/meshes/apriltag_36h11/tag36_11_0001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 scale=0.075 0.075 1.
- link tag36_11_00013: geometry visual mesh filename=package://gerard_bauzil/meshes/apriltag_36h11/tag36_11_0001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 scale=0.075 0.075 1.

File: urdf/plank_of_wood2.urdf (robot description, URDF)
Before this commit: robot plank_of_wood2, 5 links, 4 joints
Links:
- link tag36_11_00020: geometry visual mesh filename=package://gerard_bauzil/meshes/apriltag_36h11/tag36_11_0002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 scale=0.075 0.075 1.
- link tag36_11_00021: geometry visual mesh filename=package://gerard_bauzil/meshes/apriltag_36h11/tag36_11_0002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 scale=0.075 0.075 1.
- link tag36_11_00022: geometry visual mesh filename=package://gerard_bauzil/meshes/apriltag_36h11/tag36_11_0002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 scale=0.075 0.075 1.
- link tag36_11_00023: geometry visual mesh filename=package://gerard_bauzil/meshes/apriltag_36h11/tag36_11_0002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 scale=0.075 0.075 1.

File: urdf/plank_of_wood3.urdf (robot description, URDF)
Before this commit: robot plank_of_wood3, 5 links, 4 joints
Links:
- link tag36_11_00030: geometry visual mesh filename=package://gerard_bauzil/meshes/apriltag_36h11/tag36_11_0003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 scale=0.075 0.075 1.
- link tag36_11_00031: geometry visual mesh filename=package://gerard_bauzil/meshes/apriltag_36h11/tag36_11_0003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 scale=0.075 0.075 1.
- link tag36_11_00032: geometry visual mesh filename=package://gerard_bauzil/meshes/apriltag_36h11/tag36_11_0003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 scale=0.075 0.075 1.
- link tag36_11_00033: geometry visual mesh filename=package://gerard_bauzil/meshes/apriltag_36h11/tag36_11_0003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 scale=0.075 0.075 1.

File: urdf/plank_of_wood4.urdf (robot description, URDF)
Before this commit: robot plank_of_wood4, 5 links, 4 joints
Links:
- link tag36_11_00040: geometry visual mesh filename=package://gerard_bauzil/meshes/apriltag_36h11/tag36_11_0004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 scale=0.075 0.075 1.
- link tag36_11_00041: geometry visual mesh filename=package://gerard_bauzil/meshes/apriltag_36h11/tag36_11_0004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 scale=0.075 0.075 1.
- link tag36_11_00042: geometry visual mesh filename=package://gerard_bauzil/meshes/apriltag_36h11/tag36_11_0004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 scale=0.075 0.075 1.
- link tag36_11_00043: geometry visual mesh filename=package://gerard_bauzil/meshes/apriltag_36h11/tag36_11_0004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 scale=0.075 0.075 1.

File: urdf/rolling_table.urdf (robot description, URDF)
Before this commit: robot table, 4 links, 3 joints
Links:
- link tag36_11_00010: geometry visual mesh filename=package://gerard_bauzil/meshes/apriltag_36h11/tag36_11_0001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 scale=0.075 0.075 1.
- link tag36_11_00011: geometry visual mesh filename=package://gerard_bauzil/meshes/apriltag_36h11/tag36_11_0001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 scale=0.0635 0.0635 1.

File: urdf/table_140_70_73.urdf (robot description, URDF)
Before this commit: robot table, 4 links, 3 joints
Links:
- link tag36_11_00004: geometry visual mesh filename=package://gerard_bauzil/meshes/apriltag_36h11/tag36_11_0000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 scale=0.075 0.075 1.
- link tag36_11_00005: geometry visual mesh filename=package://gerard_bauzil/meshes/apriltag_36h11/tag36_11_0000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 scale=0.075 0.075 1.

File: xacro/plank_of_wood.xacro (robot description, xacro)
@@ -1,4 +1,5 @@
 <?xml version="1.0"?>
 <robot xmlns:xacro="http://www.ros.org/wiki/xacro" name="plank_of_wood$(arg number)">
+  <xacro:include filename="apriltag.xacro"/>
   <link name="base_link">
     <visual>
@@ -12,5 +13,5 @@
     <collision>
       <geometry>
-        <box size="0.203 0.043 0.116"/>
+        <box size="0.203 0.116 0.043"/>
       </geometry>
     </collision>
@@ -21,12 +22,8 @@
   </link>
   <xacro:macro name="tag" params="number x y side *material">
-    <link name="tag36_11_000${number}">
-      <visual>
-        <geometry>
-          <box size="0.06 0.06 0.002"/>
-        </geometry>
-        <xacro:insert_block name="material" />
-      </visual>
-    </link>
+    <!-- the size 0.075 corresponds to 60mm * 10 / 8 because the DAE includes white pixels on the border.-->
+    <xacro:apriltag_36h11 name="tag36_11_000${number}"
+      id="tag36_11_000${number}"
+      size="0.075" />
     <joint name="tag36_11_000${number}_joint" type="fixed">
       <parent link="base_link"/>

Commit message: AprilTag size does not take the white border into account.

File: urdf/plank_of_wood1.urdf (robot description, URDF)
Before this commit: robot plank_of_wood1, 5 links, 4 joints
Links:
- link tag36_11_00010: geometry visual mesh filename=package://gerard_bauzil/meshes/apriltag_36h11/tag36_11_0001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 scale=0.06 0.06 1.
- link tag36_11_00011: geometry visual mesh filename=package://gerard_bauzil/meshes/apriltag_36h11/tag36_11_0001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 scale=0.06 0.06 1.
- link tag36_11_00012: geometry visual mesh filename=package://gerard_bauzil/meshes/apriltag_36h11/tag36_11_0001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 scale=0.06 0.06 1.
- link tag36_11_00013: geometry visual mesh filename=package://gerard_bauzil/meshes/apriltag_36h11/tag36_11_0001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 scale=0.06 0.06 1.

File: urdf/plank_of_wood2.urdf (robot description, URDF)
Before this commit: robot plank_of_wood2, 5 links, 4 joints
Links:
- link tag36_11_00020: geometry visual mesh filename=package://gerard_bauzil/meshes/apriltag_36h11/tag36_11_0002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 scale=0.06 0.06 1.
- link tag36_11_00021: geometry visual mesh filename=package://gerard_bauzil/meshes/apriltag_36h11/tag36_11_0002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 scale=0.06 0.06 1.
- link tag36_11_00022: geometry visual mesh filename=package://gerard_bauzil/meshes/apriltag_36h11/tag36_11_0002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 scale=0.06 0.06 1.
- link tag36_11_00023: geometry visual mesh filename=package://gerard_bauzil/meshes/apriltag_36h11/tag36_11_0002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 scale=0.06 0.06 1.

File: urdf/plank_of_wood3.urdf (robot description, URDF)
Before this commit: robot plank_of_wood3, 5 links, 4 joints
Links:
- link tag36_11_00030: geometry visual mesh filename=package://gerard_bauzil/meshes/apriltag_36h11/tag36_11_0003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 scale=0.06 0.06 1.
- link tag36_11_00031: geometry visual mesh filename=package://gerard_bauzil/meshes/apriltag_36h11/tag36_11_0003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 scale=0.06 0.06 1.
- link tag36_11_00032: geometry visual mesh filename=package://gerard_bauzil/meshes/apriltag_36h11/tag36_11_0003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 scale=0.06 0.06 1.
- link tag36_11_00033: geometry visual mesh filename=package://gerard_bauzil/meshes/apriltag_36h11/tag36_11_0003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 scale=0.06 0.06 1.

File: urdf/plank_of_wood4.urdf (robot description, URDF)
Before this commit: robot plank_of_wood4, 5 links, 4 joints
Links:
- link tag36_11_00040: geometry visual mesh filename=package://gerard_bauzil/meshes/apriltag_36h11/tag36_11_0004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 scale=0.06 0.06 1.
- link tag36_11_00041: geometry visual mesh filename=package://gerard_bauzil/meshes/apriltag_36h11/tag36_11_0004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 scale=0.06 0.06 1.
- link tag36_11_00042: geometry visual mesh filename=package://gerard_bauzil/meshes/apriltag_36h11/tag36_11_0004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 scale=0.06 0.06 1.
- link tag36_11_00043: geometry visual mesh filename=package://gerard_bauzil/meshes/apriltag_36h11/tag36_11_0004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 scale=0.06 0.06 1.

File: urdf/rolling_table.urdf (robot description, URDF)
Before this commit: robot table, 4 links, 3 joints
Links:
- link tag36_11_00010: geometry visual mesh filename=package://gerard_bauzil/meshes/apriltag_36h11/tag36_11_0001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 scale=0.060 0.060 1.
- link tag36_11_00011: geometry visual mesh filename=package://gerard_bauzil/meshes/apriltag_36h11/tag36_11_0001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 scale=0.060 0.060 1.

File: urdf/table_140_70_73.urdf (robot description, URDF)
Before this commit: robot table, 4 links, 3 joints
Links:
- link tag36_11_00004: geometry visual mesh filename=package://gerard_bauzil/meshes/apriltag_36h11/tag36_11_0000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 scale=0.060 0.060 1.
- link tag36_11_00005: geometry visual mesh filename=package://gerard_bauzil/meshes/apriltag_36h11/tag36_11_0000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 scale=0.060 0.060 1.

File: xacro/apriltag.xacro (robot description, xacro)
@@ -2,4 +2,5 @@
 <robot xmlns:xacro="http://www.ros.org/wiki/xacro" name="apriltag">
   <xacro:arg name="make_urdf" default="false"/>
+  <!-- param size: size of the April tag in meters, excluding the white border. -->
   <xacro:macro name="apriltag_36h11" params="name id size">
     <link name="${name}">

File: xacro/plank_of_wood.xacro (robot description, xacro)
@@ -22,8 +22,7 @@
   </link>
   <xacro:macro name="tag" params="number x y side *material">
-    <!-- the size 0.075 corresponds to 60mm * 10 / 8 because the DAE includes white pixels on the border.-->
     <xacro:apriltag_36h11 name="tag36_11_000${number}"
       id="tag36_11_000${number}"
-      size="0.075" />
+      size="0.060" />
     <joint name="tag36_11_000${number}_joint" type="fixed">
       <parent link="base_link"/>
@@ -61,8 +60,8 @@
   <xacro:tags number="$(arg number)" x="$(arg x)" y="$(arg y)" />
   <!-- args are :
-         1 62.625 6.25
-         2 62.875 8.625
-         3 63     10.5
-         4 63.25  7.75
+         number:=1 x:=62.625 y:=6.25
+         number:=2 x:=62.875 y:=8.625
+         number:=3 x:=63     y:=10.5
+         number:=4 x:=63.25  y:=7.75
   -->
 </robot>
