Commit message: Some update

File: urdf/gerard_bauzil.urdf (robot description, URDF)
Before this commit: robot gerard_bauzil, 2 links, 1 joints
Links:
- removed link dummy
- added link world
- link base_link: mass 0.01 -> 100.00; geometry collision mesh filename=package://gerard_bauzil/wall_laas15.dae; visual mesh filename=package://gerard_bauzil/wall_laas15.dae
Joints:
- removed joint dummy_joint
- added joint world_joint: type fixed, parent world, child base_link, origin xyz=0.0 0.0 0.0 rpy=0.0 0.0 0.0

Commit message: Finish simulation with salle Gerard Bauzil

File: urdf/gerard_bauzil.urdf (robot description, URDF)
Before this commit: robot gerard_bauzil, 2 links, 1 joints
Links:
- removed link world
- link base_link: geometry collision mesh filename=package://gerard_bauzil/wall_laas15_without_floor.dae; visual mesh filename=package://gerard_bauzil/wall_laas15_without_floor.dae
Joints:
- removed joint world_joint
