Commit message: Fix orientation of tags on rolling table.

File: urdf/rolling_table.urdf (robot description, URDF)
Before this commit: robot table, 4 links, 3 joints
Joints:
- joint tag36_11_00010_joint: origin xyz=0.202 0.0075 0.75 rpy=0 0 0 -> xyz=0.202 0.0075 0.75 rpy=0 0 -1.5707963267948966
- joint tag36_11_00011_joint: origin xyz=-0.199 -0.256 0.75 rpy=0 0 0 -> xyz=-0.199 -0.256 0.75 rpy=0 0 -1.5707963267948966

Commit message: Fix table models
  - remove useless extra link and joint,
  - make rolling table 75cm high.

File: urdf/rolling_table.urdf (robot description, URDF)
Before this commit: robot table, 4 links, 3 joints
Links:
- removed link base_link
Joints:
- removed joint table_joint

File: urdf/table_140_70_73.urdf (robot description, URDF)
Before this commit: robot table, 4 links, 3 joints
Links:
- removed link base_link
Joints:
- removed joint table_joint

Commit message: [table] Rename table_link -> base_link.

File: urdf/rolling_table.urdf (robot description, URDF)
Before this commit: robot table, 3 links, 2 joints
Links:
- removed link table_link
- added link base_link, mass 2.2; collision box size=.07 .02 .63; collision box size=.07 .02 .63
Joints:
- joint tag36_11_00010_joint: parent table_link -> base_link
- joint tag36_11_00011_joint: parent table_link -> base_link

File: urdf/table_140_70_73.urdf (robot description, URDF)
Before this commit: robot table, 3 links, 2 joints
Links:
- removed link table_link
- added link base_link, mass 2.2; collision box size=.02 .02 .72; collision box size=.02 .02 .72
Joints:
- joint tag36_11_00004_joint: parent table_link -> base_link
- joint tag36_11_00005_joint: parent table_link -> base_link
