Commit message: Remove weight of driller.

File: urdf/driller.urdf (robot description, URDF)
Before this commit: robot driller, 3 links, 2 joints
Links:
- link base_link: mass 2.2 -> 0.001

File: urdf/driller_with_qr_drill.urdf (robot description, URDF)
Before this commit: robot driller, 5 links, 4 joints
Links:
- link base_link: mass 2.2 -> 0.001

File: xacro/driller_with_qr_drill.xacro (robot description, xacro)
@@ -19,7 +19,7 @@
     </collision>
     <inertial>
-      <mass value="2.2"/>
+      <mass value="0.001"/>
       <origin xyz="0 0 0" rpy="0 0 0"/>
-      <inertia ixx="0.1"  ixy="0"  ixz="0" iyy="0.1" iyz="0" izz="0.1" />
+      <inertia ixx="0.001"  ixy="0"  ixz="0" iyy="0.001" iyz="0" izz="0.001" />
     </inertial>
   </link>
