Commit message: Add SRDF + fix qt_drill model.

File: urdf/driller_with_qr_drill.urdf (robot description, URDF)
Before this commit: robot driller, 5 links, 4 joints
Links:
- link drill_link: geometry collision cylinder length=0.074 radius=0.005; visual cylinder length=0.074 radius=0.005

File: xacro/qr_drill.xacro (robot description, xacro)
@@ -14,5 +14,5 @@
       <collision>
         <geometry name="drill">
-          <cylinder length="0.05" radius="0.005"/>
+          <cylinder length="0.074" radius="0.005"/>
         </geometry>
       </collision>

Commit message: Driller uses tag 230

File: urdf/driller_with_qr_drill.urdf (robot description, URDF)
Before this commit: robot driller, 5 links, 4 joints
Links:
- removed link tag36_11_00010
- added link tag36_11_00230; visual mesh filename=package://gerard_bauzil/meshes/apriltag_36h11/tag36_11_0023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 scale=0.04 0.04 1.
Joints:
- joint tag_joint: child tag36_11_00010 -> tag36_11_00230

File: xacro/driller_with_qr_drill.xacro (robot description, xacro)
@@ -24,5 +24,5 @@
     </inertial>
   </link>
-  <xacro:qr_drill number="_00010" size="0.04" />
+  <xacro:qr_drill number="_00230" size="0.04" />
   <!-- The drill penetrates in the driller of 74 - 46.5 = 27.5mm -->
   <joint name="drill_joint" type="fixed">

Commit message: Update tag size on driller.

File: urdf/driller_with_qr_drill.urdf (robot description, URDF)
Before this commit: robot driller, 5 links, 4 joints
Links:
- link tag36_11_00230: geometry visual mesh filename=package://gerard_bauzil/meshes/apriltag_36h11/tag36_11_0023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 scale=0.064 0.064 1.

File: xacro/driller_with_qr_drill.xacro (robot description, xacro)
@@ -24,5 +24,5 @@
     </inertial>
   </link>
-  <xacro:qr_drill number="_00230" size="0.04" />
+  <xacro:qr_drill number="_00230" size="0.064" />
   <!-- The drill penetrates in the driller of 74 - 46.5 = 27.5mm -->
   <joint name="drill_joint" type="fixed">

File: xacro/qr_drill.xacro (robot description, xacro)
@@ -2,5 +2,5 @@
 <robot xmlns:xacro="http://www.ros.org/wiki/xacro" name="qr_drill">
   <xacro:include filename="apriltag.xacro"/>
-  <xacro:macro name="qr_drill" params="number size:=0.04">
+  <xacro:macro name="qr_drill" params="number size:=0.064">
     <link name="drill_link">
       <visual>

Commit message: Add collision model for the tag of driller_with_qr_drill.urdf

File: urdf/driller_with_qr_drill.urdf (robot description, URDF)
Before this commit: robot driller, 5 links, 4 joints
Links:
- link tag36_11_00230: geometry collision box size=0.08 0.08 0.0001; visual mesh filename=package://gerard_bauzil/meshes/apriltag_36h11/tag36_11_0023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 scale=0.064 0.064 1.

Commit message: add tag230 to the back

File: urdf/driller_with_qr_drill.urdf (robot description, URDF)
Before this commit: robot driller, 5 links, 4 joints
Links:
- added link tag36_11_00230; visual mesh filename=package://gerard_bauzil/meshes/apriltag_36h11/tag36_11_0023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 scale=0.04 0.04 1.
- added link tag_support_link_back, mass 0.001; collision mesh filename=package://gerard_bauzil/meshes/driller/qr_drill_back.stl; visual mesh filename=package://gerard_bauzil/meshes/driller/qr_drill_back.stl
Joints:
- added joint tag_joint_back: type fixed, parent tag_support_link_back, child tag36_11_00230, origin xyz=0 0 0.002
- added joint tag_support_joint_back: type fixed, parent drill_link, child tag_support_link_back, origin xyz=-0.0 0.00 -0.22 rpy=3.141592653589793 0 -1.57079632679

File: xacro/driller_with_qr_drill.xacro (robot description, xacro)
@@ -24,6 +24,6 @@
     </inertial>
   </link>
-  <!-- <xacro:qr_drill number="_00230" size="0.064" /> -->
-  <xacro:qr_drill number="_00023" size="0.04" />
+  <xacro:qr_drill number="_00230" size="0.04" />
+  <!-- <xacro:qr_drill number="_00023" size="0.04" /> -->
   <!-- The drill penetrates in the driller of 74 - 46.5 = 27.5mm -->
   <joint name="drill_joint" type="fixed">

File: xacro/qr_drill.xacro (robot description, xacro)
@@ -46,4 +46,23 @@
       </inertial>
     </link>
+    <link name="tag_support_link_back">
+      <visual>
+        <geometry>
+          <mesh filename="package://gerard_bauzil/meshes/driller/qr_drill_back.stl"/>
+        </geometry>
+        <material name="blue">
+          <color rgba="0.1 0.1 0.9 1"/>
+        </material>
+      </visual>
+      <collision>
+        <geometry>
+          <mesh filename="package://gerard_bauzil/meshes/driller/qr_drill_back.stl"/>
+        </geometry>
+      </collision>
+      <inertial>
+        <mass value="0.001"/>
+        <inertia ixx="0.001"  ixy="0"  ixz="0" iyy="0.001" iyz="0" izz="0.001" />
+      </inertial>
+    </link>
     <joint name="tag_support_joint" type="fixed">
       <parent link="drill_link"/>
@@ -53,8 +72,21 @@
       <!-- <origin xyz="0 0.049 0.041" rpy="0 3.141592653589793 0" /> -->
     </joint>
-    <xacro:apriltag_36h11 name="tag36_11${number}" id="tag36_11${number}" size="${size}" />
+     <joint name="tag_support_joint_back" type="fixed">
+      <parent link="drill_link"/>
+      <child  link="tag_support_link_back"/>
+      <!-- 74mm / 2 + 4mm -->
+      <origin xyz="-0.0 0.00 -0.22" rpy="3.141592653589793 0 -1.57079632679" />
+      <!-- <origin xyz="0 0.049 0.041" rpy="0 3.141592653589793 0" /> -->
+    </joint>
+    <xacro:apriltag_36h11 name="tag36_11_00023" id="tag36_11_00023" size="0.04" />
+    <xacro:apriltag_36h11 name="tag36_11_00230" id="tag36_11_00230" size="0.04" />
     <joint name="tag_joint" type="fixed">
       <parent link="tag_support_link_top"/>
-      <child  link="tag36_11${number}"/>
+      <child  link="tag36_11_00023"/>
+      <origin xyz="0 0 0.002" />
+    </joint>
+     <joint name="tag_joint_back" type="fixed">
+      <parent link="tag_support_link_back"/>
+      <child  link="tag36_11_00230"/>
       <origin xyz="0 0 0.002" />
     </joint>

Commit message: done positioning tag supports and tags

File: urdf/driller_with_qr_drill.urdf (robot description, URDF)
Before this commit: robot driller, 7 links, 6 joints
Joints:
- joint tag_support_joint: origin xyz=-0.06 0.00 -0.111 rpy=3.141592653589793 0 -1.57079632679 -> xyz=-0.06 0.00 -0.105 rpy=3.141592653589793 0 -1.57079632679
- joint tag_support_joint_back: origin xyz=-0.0 0.00 -0.22 rpy=3.141592653589793 0 -1.57079632679 -> xyz=-0.0 0.00 -0.194 rpy=3.141592653589793 0 -1.57079632679

File: xacro/qr_drill.xacro (robot description, xacro)
@@ -69,5 +69,5 @@
       <child  link="tag_support_link_top"/>
       <!-- 74mm / 2 + 4mm -->
-      <origin xyz="-0.06 0.00 -0.111" rpy="3.141592653589793 0 -1.57079632679" />
+      <origin xyz="-0.06 0.00 -0.105" rpy="3.141592653589793 0 -1.57079632679" />
       <!-- <origin xyz="0 0.049 0.041" rpy="0 3.141592653589793 0" /> -->
     </joint>
@@ -76,5 +76,5 @@
       <child  link="tag_support_link_back"/>
       <!-- 74mm / 2 + 4mm -->
-      <origin xyz="-0.0 0.00 -0.22" rpy="3.141592653589793 0 -1.57079632679" />
+      <origin xyz="-0.0 0.00 -0.194" rpy="3.141592653589793 0 -1.57079632679" />
       <!-- <origin xyz="0 0.049 0.041" rpy="0 3.141592653589793 0" /> -->
     </joint>

Commit message: Changes

File: urdf/driller_with_qr_drill.urdf (robot description, URDF)
Before this commit: robot driller, 7 links, 6 joints
Joints:
- joint tag_joint: origin xyz=0 0 0.002 -> xyz=0.002 0.042 0.002 rpy=0 0 0
- joint tag_joint_back: origin xyz=0 0 0.002 -> xyz=0 -0.00 0.0002
- joint tag_support_joint: origin xyz=-0.06 0.00 -0.105 rpy=3.141592653589793 0 -1.57079632679 -> xyz=-0.052 0.00 -0.10 rpy=3.141592653589793 0.0 -1.57079632679

File: xacro/qr_drill.xacro (robot description, xacro)
@@ -69,5 +69,5 @@
       <child  link="tag_support_link_top"/>
       <!-- 74mm / 2 + 4mm -->
-      <origin xyz="-0.06 0.00 -0.105" rpy="3.141592653589793 0 -1.57079632679" />
+      <origin xyz="-0.066 0.00 -0.100" rpy="3.141592653589793 0 -1.57079632679" />
       <!-- <origin xyz="0 0.049 0.041" rpy="0 3.141592653589793 0" /> -->
     </joint>
