Commit message: Fix SRDF of rolling_table and plank_of_wood_srdf

File: xacro/plank_of_wood_srdf.xacro (robot description, xacro)
@@ -2,9 +2,17 @@
 <robot xmlns:xacro="http://www.ros.org/wiki/xacro" name="plank_of_wood$(arg number)">
   <handle name="handle1" clearance="0.08">
-    <position>  0.1015 0 0  0 0 0 1 </position>
+    <position> -0.06 0 0  0.707106781187 -0.707106781187 0 0 </position>
     <link name="base_link"/>
   </handle>
   <handle name="handle2" clearance="0.08">
-    <position> -0.1015 0 0  0 0 0 1 </position>
+    <position> 0.06 0 0  0 0 -0.707106781187 0.707106781187 </position>
+    <link name="base_link"/>
+  </handle>
+  <handle name="handle3" clearance="0.08">
+    <position> -0.06 0 0  0.707106781187 0.707106781187 0 0 </position>
+    <link name="base_link"/>
+  </handle>
+  <handle name="handle4" clearance="0.08">
+    <position> 0.06 0 0  0 0 0.707106781187 0.707106781187 </position>
     <link name="base_link"/>
   </handle>
@@ -12,8 +20,44 @@
     <link name="base_link"/>
     <point>
-      +0.102 +0.022 -0.058
-      +0.102 -0.022 -0.058
-      -0.102 -0.022 -0.058
-      -0.102 +0.022 -0.058
+      +0.105 -0.071 +0.02
+      +0.105 -0.071 -0.02
+      -0.105 -0.071 -0.02
+      -0.105 -0.071 +0.02
+    </point>
+    <shape>
+      4 3 2 1 0
+    </shape>
+  </contact>
+  <contact name="top_surface">
+    <link name="base_link"/>
+    <point>
+      +0.1015 0.058 +0.022
+      +0.1015 0.058 -0.022
+      -0.1015 0.058 -0.022
+      -0.1015 0.058 +0.022
+    </point>
+    <shape>
+      4 0 1 2 3
+    </shape>
+  </contact>
+  <contact name="front_surface">
+    <link name="base_link"/>
+    <point>
+      +0.1015 +0.058 +0.022
+      +0.1015 +0.058 -0.022
+      +0.1015 -0.058 -0.022
+      +0.1015 -0.058 +0.022
+    </point>
+    <shape>
+      4 3 2 1 0
+    </shape>
+  </contact>
+  <contact name="rear_surface">
+    <link name="base_link"/>
+    <point>
+      -0.1015 +0.058 +0.022
+      -0.1015 +0.058 -0.022
+      -0.1015 -0.058 -0.022
+      -0.1015 -0.058 +0.022
     </point>
     <shape>
