Commit message: change the driller qr support to top

File: xacro/driller_with_qr_drill.urdf (robot description, URDF)
Before this commit: robot driller, 5 links, 4 joints
Joints:
- joint tag_support_joint: origin xyz=-0.06 0.00 -0.111 rpy=3.141592653589793 0 -1.57079632679 -> xyz=0.06 0.00 -0.111 rpy=3.141592653589793 1.57079632679 0

File: xacro/driller_with_qr_drill.xacro (robot description, xacro)
@@ -24,5 +24,6 @@
     </inertial>
   </link>
-  <xacro:qr_drill number="_00230" size="0.064" />
+  <!-- <xacro:qr_drill number="_00230" size="0.064" /> -->
+  <xacro:qr_drill number="_00023" size="0.04" />
   <!-- The drill penetrates in the driller of 74 - 46.5 = 27.5mm -->
   <joint name="drill_joint" type="fixed">

File: xacro/qr_drill.xacro (robot description, xacro)
@@ -2,5 +2,5 @@
 <robot xmlns:xacro="http://www.ros.org/wiki/xacro" name="qr_drill">
   <xacro:include filename="apriltag.xacro"/>
-  <xacro:macro name="qr_drill" params="number size:=0.064">
+  <xacro:macro name="qr_drill" params="number size:=0.040">
     <link name="drill_link">
       <visual>
@@ -27,8 +27,8 @@
       </collision_checking>
     </link>
-    <link name="tag_support_link">
+    <link name="tag_support_link_top">
       <visual>
         <geometry>
-          <mesh filename="package://gerard_bauzil/meshes/driller/qr_drill.stl"/>
+          <mesh filename="package://gerard_bauzil/meshes/driller/qr_drill_top.stl"/>
         </geometry>
         <material name="blue">
@@ -38,5 +38,5 @@
       <collision>
         <geometry>
-          <mesh filename="package://gerard_bauzil/meshes/driller/qr_drill.stl"/>
+          <mesh filename="package://gerard_bauzil/meshes/driller/qr_drill_top.stl"/>
         </geometry>
       </collision>
@@ -48,13 +48,14 @@
     <joint name="tag_support_joint" type="fixed">
       <parent link="drill_link"/>
-      <child  link="tag_support_link"/>
+      <child  link="tag_support_link_top"/>
       <!-- 74mm / 2 + 4mm -->
-      <origin xyz="0 0.049 0.041" rpy="0 3.141592653589793 0" />
+      <origin xyz="-0.06 0.00 -0.111" rpy="3.141592653589793 0 -1.57079632679" />
+      <!-- <origin xyz="0 0.049 0.041" rpy="0 3.141592653589793 0" /> -->
     </joint>
     <xacro:apriltag_36h11 name="tag36_11${number}" id="tag36_11${number}" size="${size}" />
     <joint name="tag_joint" type="fixed">
-      <parent link="tag_support_link"/>
+      <parent link="tag_support_link_top"/>
       <child  link="tag36_11${number}"/>
-      <origin xyz="0 0 0.0022" />
+      <origin xyz="0 0 0.002" />
     </joint>
   </xacro:macro>
